Commit message: Feat: Corrections on RViz

File: eboat_description/urdf/eboat copy.urdf (robot description, URDF)
Before this commit: robot eboat4, 23 links, 22 joints
Joints:
- removed joint sail_joint
- added joint sail_joint_2: type fixed, parent boom_link, child rope_c_link, origin xyz=-1.7978 0 0.0223 rpy=1.5708 0 0

Commit message: Feat: Lidar

File: eboat_description/urdf/eboat copy.urdf (robot description, URDF)
Before this commit: robot eboat4, 23 links, 22 joints
Joints:
- removed joint sail_joint_2
- added joint sail_joint: type fixed, parent boom_link, child rope_c_link, origin xyz=-1.7978 0 0.0223 rpy=1.5708 0 0

File: eboat_description/urdf/eboat4tr.urdf.xacro (robot description, xacro)
@@ -230,5 +230,5 @@
         </inertial>
     </link>
-    <joint name="propeller_joint" type="revolute">
+    <joint name="propeller_joint" type="continuous">
         <origin xyz="-0.089683 -7.7043e-18 -0.949" rpy="-1.26162e-16 -0 0" />
         <parent link="eletric_engine_link" />
@@ -294,4 +294,52 @@
         <child link="camera_bow_link" />
     </joint>
+         <!-- LIDAR Sensor -->
+        <link name="lidar_link">
+            <visual>
+            <geometry>
+                <cylinder length="0.5" radius="0.05"/>
+            </geometry>
+            <origin xyz="0 0 0" rpy="0 0 0"/>
+            <material name="blue"/>
+            </visual>
+            <inertial>
+            <origin xyz="0 0 0" rpy="0 0 0"/>
+            <mass value="0.1"/>
+            <inertia ixx="1.0" ixy="2.0" ixz="0" iyy="1.0" iyz="0" izz="1.0"/>
+            </inertial>
+        </link>
+        <!-- Attach the LIDAR sensor to the boat -->
+        <joint name="lidar_joint" type="fixed">
+            <parent link="base_link"/>
+            <child link="lidar_link"/>
+            <origin xyz="1 0 0.75" rpy="0 0 0"/>
+        </joint>
+    <!-- LIDAR Gazebo plugin -->
+    <gazebo reference="lidar_link">
+        <sensor type="ray" name="lidar">
+            <pose>0 0 0 0 0 0</pose>
+            <visualize>true</visualize>
+            <update_rate>10</update_rate>
+            <ray>
+                <scan>
+                    <horizontal>
+                        <samples>360</samples>
+                        <resolution>1</resolution>
+                        <min_angle>-1.5708</min_angle> <!-- -pi/2 radian -->
+                        <max_angle>1.5708</max_angle> <!-- pi/2 radian -->
+                    </horizontal>
+                </scan>
+                <range>
+                    <min>0.1</min>
+                    <max>10</max>
+                    <resolution>0.01</resolution>
+                </range>
+            </ray>
+            <plugin name="gazebo_ros_head_hokuyo_controller" filename="libgazebo_ros_laser.so">
+                <topicName>/lidar_scan</topicName>
+                <frameName>lidar_link</frameName>
+            </plugin>
+        </sensor>
+    </gazebo>
     <!--COLORS-->
     <gazebo reference="boom_link">

File: eboat_description/urdf/modified_urdf.urdf (robot description, URDF)
Before this commit: robot eboat4, 23 links, 22 joints
Links:
- removed link base_link
- added link map
- link camera_link: geometry collision box size=0.1 0.1 0.1; visual box size=0.1 0.1 0.1
- link lidar_link: geometry collision cylinder length=0.2 radius=0.05; visual cylinder length=0.2 radius=0.05
Joints:
- removed joint sail_joint_2
- added joint sail_joint: type fixed, parent boom_link, child rope_c_link, origin xyz=-1.7978 0 0.0223 rpy=1.5708 0 0
- joint camera_top_joint: origin xyz=-0.053 0 3.765 rpy=0 0 0 -> xyz=0.053 0 -2.832 rpy=0 0 0

File: eboat_gazebo/worlds/ocean_RL_training.world.xacro (robot description, xacro)
@@ -10,4 +10,9 @@
             <uri>$(find eboat_description)/models/wayPointMarker</uri>
         </include>
+        <include>
+            <name>buoy_red</name>
+            <pose>10 0 0 0 0 0 0</pose>
+            <uri>$(find eboat_description)/models/buoy_red</uri>
+        </include>
         <!--PHYSICS ENGINE-->
         <physics type="ode">
@@ -18,5 +23,5 @@
             </ode>
             <max_step_size>0.01</max_step_size>
-            <real_time_update_rate>0</real_time_update_rate>
+            <real_time_update_rate>100</real_time_update_rate>
         </physics>
     </world>
