Commit message: Feat: Raycast configuration

File: eboat_description/urdf/eboat4tr.urdf copy.xacro (robot description, xacro)
@@ -312,71 +312,84 @@
         <material>Gazebo/Grey</material>
     </gazebo>
-<!-- RAY SENSOR Link -->
-    <link name="ray_link">
-        <visual>
-            <origin xyz="-2.03098 6.90927e-15 -0.125" rpy="0 -0 0" />
-            <geometry>
-                <box size="2 0 0"/>
-            </geometry>
-        </visual>
-        <collision>
-            <origin xyz="-2.03098 6.90927e-15 -0.125" rpy="0 -0 0" />
-            <geometry>
-                <box size="2 0 0"/>
-            </geometry>
-        </collision>
-        <inertial>
-            <mass value="0.001" />
-            <inertia ixx="0.0001" ixy="0.0" ixz="0.0" iyy="0.0001" iyz="0.0" izz="0.0001" />
-        </inertial>
-    </link>
-    <!--RAY SENSOR joint-->
-    <joint name="ray_joint" type="fixed">
-        <origin xyz="0 0 0.6" rpy="0 0 0" />
-        <parent link="camera_bow_link" />
-        <child link="ray_link" />
-    </joint>
-<!--RAY SENSOR liked on camera link-->
-    <gazebo reference="ray_link">
-        <sensor type="ray" name="camera_bow_sensor">
+<!-- LIDAR Sensor link -->
+<!--     <link name="eboat_lidar_link">
+        <visual>
+            <origin xyz="0 0 0" rpy="0 0 0" />
+            <geometry>
+                <cylinder length="0.5" radius="0.08"/>
+            </geometry>
+        </visual>
+        <collision>
+            <origin xyz="0 0 0" rpy="0 0 0" />
+            <geometry>
+                <cylinder length="0.5" radius="0.8"/>
+            </geometry>
+        </collision>
+        <inertial>
+            <origin xyz="0 0 0" rpy="0 0 0"/>
+            <mass value="0.1" />
+            <inertia ixx="0.1" ixy="0.0" ixz="0.0" iyy="0.1" iyz="0.0" izz="0.1" />
+        </inertial>
+    </link> -->
+<!-- Attach the LIDAR sensor to the boat -->
+        <!-- <joint name="eboat_lidar_joint" type="fixed">
+            <parent link="base_link"/>
+            <child link="eboat_lidar_link"/>
+            <origin xyz="1 0 0.75" rpy="0 0 0"/>
+        </joint> -->
+<!-- Attach the LIDAR sensor to the boat -->
+ <!-- <sensor type="ray" name="eboat_lidar_sensor_visual">
+            <pose>0 0 0 0 0 0</pose>
             <visualize>true</visualize>
-            <material>Gazebo/Blue</material>
-            <contact>
-                <collide>true</collide>
-                    <collide_without_contact>true</collide_without_contact>
-                    <collide_bitmask>0x02</collide_bitmask>
-                    <collide_without_contact_bitmask>0x01</collide_without_contact_bitmask>
-            </contact>
-            <visualize>true</visualize>
-            <update_rate>1</update_rate>
-            <ray>
-                <scan>
-                    <horizontal>
-                        <samples>120</samples>
-                        <resolution>1</resolution>
-                        <min_angle>-1.05</min_angle>
-                        <max_angle>1.05</max_angle>
-                    </horizontal>
-                </scan>
-                <range>
-                    <min>0.1</min>
-                    <max>40.0</max>
-                    <resolution>0.1</resolution>
-                 </range>
-                    <noise>
-                    <type>gaussian</type>
-                    <!-- Noise parameters based on published spec for Hokuyo laser
-                        achieving "+-30mm" accuracy at range < 10m.  A mean of 0.0m and
-                        stddev of 0.01m will put 99.7% of samples within 0.03m of the true
-                        reading. -->
-                    <mean>0.0</mean>
-                    <stddev>0.01</stddev>
-                    </noise>
-                </ray>
-                <plugin name="gazebo_ros_camera_bow_controller" filename="libgazebo_ros_laser.so">
-                    <topicName>/eboat/camera_bow/scan</topicName>
-                    <frameName>ray_link</frameName>
-                </plugin>
-            </sensor>
-        </gazebo>
+            <update_rate>10</update_rate>
+            <geometry>
+                <cylinder length="0.5" radius="0.8"/>
+            </geometry>
+            <material>
+                <ambient>0 0 1 1</ambient>
+            </material>
+            <origin xyz="0 0 0" rpy="0 0 0"/>
+    </sensor> -->
+<!--RAY SENSOR-->
+<gazebo reference="camera_link">
+    <sensor type="ray" name="head_hokuyo_sensor">
+        <material>Gazebo/Blue</material>
+        <contact>
+                <collide_without_contact>true</collide_without_contact>
+                <collide_bitmask>0x02</collide_bitmask>
+                <collide_without_contact_bitmask>0x01</collide_without_contact_bitmask>
+        </contact>
+        <pose>0 0 0 0 0 0</pose>
+        <visualize>true</visualize>
+        <update_rate>10</update_rate>
+        <ray>
+            <scan>
+                <horizontal>
+                    <samples>120</samples>
+                    <resolution>1</resolution>
+                    <min_angle>-1.05</min_angle>
+                    <max_angle>1.05</max_angle>
+                </horizontal>
+            </scan>
+            <range>
+                <min>0.1</min>
+                <max>40.0</max>
+                <resolution>0.1</resolution>
+             </range>
+                <noise>
+                <type>gaussian</type>
+                <!-- Noise parameters based on published spec for Hokuyo laser
+                    achieving "+-30mm" accuracy at range < 10m.  A mean of 0.0m and
+                    stddev of 0.01m will put 99.7% of samples within 0.03m of the true
+                    reading. -->
+                <mean>0.0</mean>
+                <stddev>0.01</stddev>
+                </noise>
+            </ray>
+            <plugin name="gazebo_ros_head_hokuyo_controller" filename="libgazebo_ros_laser.so">
+                <topicName>/eboat/laser/scan</topicName>
+                <frameName>camera_link</frameName>
+            </plugin>
+        </sensor>
+    </gazebo>
 </robot>

File: eboat_gazebo/worlds/empty_ocean.world.xacro (robot description, xacro)
@@ -9,4 +9,19 @@
       <xacro:include filename="$(find eboat_gazebo)/worlds/ocean.xacro" />
       <xacro:ocean />
+      <include>
+            <name>buoy_red</name>
+            <pose>15 5 0 0 0 0 0</pose>
+            <uri>$(find eboat_description)/models/buoy_red</uri>
+        </include>
+        <include>
+            <name>buoy_green</name>
+            <pose>15.0 0.0 0 0 0 0 0</pose>
+            <uri>$(find eboat_description)/models/buoy_green</uri>
+        </include>
+        <include>
+            <name>buoy_yellow</name>
+            <pose>-20.0 10.0 0 0 0 0 0</pose>
+            <uri>$(find eboat_description)/models/buoy_yellow</uri>
+        </include>
       <!--PHYSICS ENGINE-->
         <physics type="ode">

File: eboat_gazebo/worlds/ocean_RL_training.world.xacro (robot description, xacro)
@@ -15,4 +15,19 @@
             <uri>$(find eboat_description)/models/wayPointMarker</uri>
         </include>
+        <include>
+            <name>buoy_red</name>
+            <pose>15 5 0 0 0 0 0</pose>
+            <uri>$(find eboat_description)/models/buoy_red</uri>
+        </include>
+        <include>
+            <name>buoy_green</name>
+            <pose>15.0 0.0 0 0 0 0 0</pose>
+            <uri>$(find eboat_description)/models/buoy_green</uri>
+        </include>
+        <include>
+            <name>buoy_yellow</name>
+            <pose>-20.0 10.0 0 0 0 0 0</pose>
+            <uri>$(find eboat_description)/models/buoy_yellow</uri>
+        </include>
         <!--PHYSICS ENGINE-->
         <physics type="ode">
@@ -23,5 +38,5 @@
             </ode>
             <max_step_size>0.01</max_step_size>
-            <real_time_update_rate>0</real_time_update_rate>
+            <real_time_update_rate>30</real_time_update_rate>
         </physics>
     </world>
