Commit message: New gymnasium environment where it is possible to execute multiple instances of the E-Boat.

File: eboat_description/urdf/eboat4tr.urdf.xacro (robot description, xacro)
@@ -234,6 +234,6 @@
         <parent link="eletric_engine_link" />
         <child link="propeller_link" />
-        <axis xyz="0 0 1"/>
-        <limit effort="1" velocity="20" />
+        <axis xyz="1 0 0"/>
+        <limit effort="1000" velocity="20" />
         <joint_properties friction="0.0"/>
     </joint>

File: eboat_gazebo/worlds/empty_ocean.world.xacro (robot description, xacro)
@@ -17,5 +17,5 @@
           </ode>
           <max_step_size>0.01</max_step_size>
-          <real_time_update_rate>100.0</real_time_update_rate>
+          <real_time_update_rate>0</real_time_update_rate>
       </physics>
     </world>

Commit message: Feat: New avoindece obstacles

File: eboat_description/urdf/eboat4tr.urdf.xacro (robot description, xacro)
@@ -297,4 +297,58 @@
         <child link="camera_bow_link" />
     </joint>
+        <!-- LIDAR Sensor -->
+        <link name="lidar_link">
+            <visual>
+            <geometry>
+                <cylinder length="0.5" radius="0.05"/>
+            </geometry>
+            <origin xyz="0 0 0" rpy="0 0 0"/>
+            <material name="blue"/>
+            </visual>
+        <inertial>
+                <origin xyz="0 0 0" rpy="0 0 0"/>
+                <mass value="0.1"/>
+                <inertia ixx="0.0001" ixy="0" ixz="0" iyy="0.0001" iyz="0" izz="0.0001"/>
+            </inertial>
+        </link>
+        <!-- Attach the LIDAR sensor to the boat -->
+        <joint name="lidar_joint" type="fixed">
+            <parent link="base_link"/>
+            <child link="lidar_link"/>
+            <origin xyz="1 0 0.75" rpy="0 0 0"/>
+        </joint>
+        <!-- LIDAR Gazebo plugin -->
+        <gazebo reference="lidar_link">
+        <material>Gazebo/Grey</material>
+            <contact>
+                <collide_without_contact>true</collide_without_contact>
+                <collide_bitmask>0x02</collide_bitmask>
+                <collide_without_contact_bitmask>0x01</collide_without_contact_bitmask>
+            </contact>
+        <sensor type="ray" name="lidar">
+            <pose>0 0 0 0 0 0</pose>
+            <visualize>true</visualize>
+            <update_rate>10</update_rate>
+            <ray>
+                <scan>
+                    <horizontal>
+                        <samples>360</samples>
+                        <resolution>1</resolution>
+                        <min_angle>-1.5708</min_angle> <!-- -pi/2 radian -->
+                        <max_angle>1.5708</max_angle> <!-- pi/2 radian -->
+                    </horizontal>
+                </scan>
+                <range>
+                    <min>0.1</min>
+                    <max>10</max>
+                    <resolution>0.01</resolution>
+                </range>
+            </ray>
+            <plugin name="gazebo_ros_head_hokuyo_controller" filename="libgazebo_ros_laser.so">
+                <topicName>/lidar_scan</topicName>
+                <frameName>lidar_link</frameName>
+            </plugin>
+        </sensor>
+        </gazebo>
     <!--COLORS-->
     <gazebo reference="boom_link">

File: eboat_gazebo/worlds/ocean_RL_training.world.xacro (robot description, xacro)
@@ -2,17 +2,78 @@
 <sdf version="1.6" xmlns:xacro="http://ros.org/wiki/xacro">
     <world name="ocean">
-        <gui fullscreen='0'>
-            <camera name='user_camera'>
-                <pose>-85.03 -3.517 26.21 0 0.212 -0.0332</pose>
-            </camera>
-        </gui>
         <xacro:include filename="$(find eboat_gazebo)/worlds/ocean.xacro" />
         <xacro:ocean />
         <!--WAYPOINT OBJECT-->
-        <include>
+       <!--  <include>
             <name>wayPointMarker</name>
-            <pose>100.0 0.0 0 0 0 0</pose>
+            <pose>0 100.0 0 0 0 0</pose>
             <uri>$(find eboat_description)/models/wayPointMarker</uri>
         </include>
+ -->
+        <include>
+            <name>buoy_red</name>
+            <pose>15 5 0 0 0 0 0</pose>
+            <uri>$(find eboat_description)/models/buoy_red</uri>
+        </include>
+        <include>
+            <name>buoy_green</name>
+            <pose>15.0 0.0 0 0 0 0 0</pose>
+            <uri>$(find eboat_description)/models/buoy_green</uri>
+        </include>
+        <include>
+            <name>buoy_yellow</name>
+            <pose>-20.0 10.0 0 0 0 0 0</pose>
+            <uri>$(find eboat_description)/models/buoy_yellow</uri>
+        </include>
+        <!-- <include>
+            <name>buoy_red1</name>
+            <pose>50 30 0 0 0 0 0</pose>
+            <uri>$(find eboat_description)/models/buoy_red</uri>
+        </include>
+         <include>
+            <name>buoy_red2</name>
+            <pose>50 40 0 0 0 0 0</pose>
+            <uri>$(find eboat_description)/models/buoy_red</uri>
+        </include>
+         <include>
+            <name>buoy_red3</name>
+            <pose>50 -10 0 0 0 0 0</pose>
+            <uri>$(find eboat_description)/models/buoy_red</uri>
+        </include>
+         <include>
+            <name>buoy_re4</name>
+            <pose>50 -30 0 0 0 0 0</pose>
+            <uri>$(find eboat_description)/models/buoy_red</uri>
+        </include>
+         <include>
+            <name>buoy_red5</name>
+            <pose>50 -50 0 0 0 0 0</pose>
+            <uri>$(find eboat_description)/models/buoy_red</uri>
+        </include>
+        <include>
+            <name>buoy_red6</name>
+            <pose>12.0 20.0 0 0 0 0 0</pose>
+            <uri>$(find eboat_description)/models/buoy_red</uri>
+        </include>
+         <include>
+            <name>buoy_red7</name>
+            <pose>100.0 -50.0 0 0 0 0 0</pose>
+            <uri>$(find eboat_description)/models/buoy_red</uri>
+        </include>
+         <include>
+            <name>buoy_red8</name>
+            <pose>110.0 -60.0 0 0 0 0 0</pose>
+            <uri>$(find eboat_description)/models/buoy_red</uri>
+        </include>
+         <include>
+            <name>buoy_red9</name>
+            <pose>80.0 -100.0 0 0 0 0 0</pose>
+            <uri>$(find eboat_description)/models/buoy_red</uri>
+        </include>
+         <include>
+            <name>buoy_red10</name>
+            <pose>95.0 -20.0 0 0 0 0 0</pose>
+            <uri>$(find eboat_description)/models/buoy_red</uri>
+        </include> -->
         <!--PHYSICS ENGINE-->
         <physics type="ode">
@@ -23,5 +84,5 @@
             </ode>
             <max_step_size>0.01</max_step_size>
-            <real_time_update_rate>0</real_time_update_rate>
+            <real_time_update_rate>30</real_time_update_rate>
         </physics>
     </world>

Commit message: Feat: 15 samples to avoindence obstacles

File: eboat_description/urdf/eboat4tr.urdf.xacro (robot description, xacro)
@@ -317,15 +317,10 @@
             <origin xyz="-2.03098 6.90927e-15 -0.125" rpy="0 -0 0" />
             <geometry>
-                <box size="2 0 0"/>
-            </geometry>
-        </visual>
-        <collision>
-            <origin xyz="-2.03098 6.90927e-15 -0.125" rpy="0 -0 0" />
-            <geometry>
-                <box size="2 0 0"/>
-            </geometry>
-        </collision>
-        <inertial>
-            <mass value="0.001" />
+                <box size="0.1 0.1 0.1"/>
+            </geometry>
+        </visual>
+        <inertial>
+            <origin xyz="0.0526688 -2.92253e-05 0.2517" rpy="0 0 0"/>
+            <mass value="0.1" />
             <inertia ixx="0.0001" ixy="0.0" ixz="0.0" iyy="0.0001" iyz="0.0" izz="0.0001" />
         </inertial>
@@ -339,13 +334,12 @@
 <!--RAY SENSOR liked on camera link-->
     <gazebo reference="ray_link">
-        <sensor type="ray" name="camera_bow_sensor">
+        <sensor type="ray" name="laser_scan">
             <visualize>true</visualize>
             <material>Gazebo/Blue</material>
-            <contact>
-                <collide>true</collide>
-                    <collide_without_contact>true</collide_without_contact>
-                    <collide_bitmask>0x02</collide_bitmask>
-                    <collide_without_contact_bitmask>0x01</collide_without_contact_bitmask>
-            </contact>
+                <contact>
+                        <collide_without_contact>true</collide_without_contact>
+                        <collide_bitmask>0x02</collide_bitmask>
+                        <collide_without_contact_bitmask>0x01</collide_without_contact_bitmask>
+                </contact>
             <visualize>true</visualize>
             <update_rate>1</update_rate>
@@ -353,5 +347,5 @@
                 <scan>
                     <horizontal>
-                        <samples>120</samples>
+                        <samples>15</samples>
                         <resolution>1</resolution>
                         <min_angle>-1.05</min_angle>
@@ -361,5 +355,5 @@
                 <range>
                     <min>0.1</min>
-                    <max>40.0</max>
+                    <max>10</max>
                     <resolution>0.1</resolution>
                  </range>
@@ -374,6 +368,6 @@
                     </noise>
                 </ray>
-                <plugin name="gazebo_ros_camera_bow_controller" filename="libgazebo_ros_laser.so">
-                    <topicName>/eboat/camera_bow/scan</topicName>
+                <plugin name="gazebo_ros_head_hokuyo_controller" filename="libgazebo_ros_laser.so">
+                    <topicName>/eboat/laser/scan</topicName>
                     <frameName>ray_link</frameName>
                 </plugin>

File: eboat_gazebo/worlds/empty_ocean.world.xacro (robot description, xacro)
@@ -11,10 +11,10 @@
       <include>
             <name>buoy_red</name>
-            <pose>15 5 0 0 0 0 0</pose>
+            <pose>35 5 0 0 0 0 0</pose>
             <uri>$(find eboat_description)/models/buoy_red</uri>
         </include>
         <include>
             <name>buoy_green</name>
-            <pose>15.0 0.0 0 0 0 0 0</pose>
+            <pose>45 0.0 0 0 0 0 0</pose>
             <uri>$(find eboat_description)/models/buoy_green</uri>
         </include>
@@ -32,5 +32,5 @@
           </ode>
           <max_step_size>0.01</max_step_size>
-          <real_time_update_rate>100</real_time_update_rate>
+          <real_time_update_rate>3000</real_time_update_rate>
       </physics>
     </world>

File: eboat_gazebo/worlds/ocean.world.xacro (robot description, xacro)
@@ -30,5 +30,5 @@
           </ode>
           <max_step_size>0.01</max_step_size>
-          <real_time_update_rate>100.0</real_time_update_rate>
+          <real_time_update_rate>3000</real_time_update_rate>
       </physics>
       <!--Wind. Note, wind parameters are set in the plugin.-->

File: eboat_gazebo/worlds/ocean_RL_training.world.xacro (robot description, xacro)
@@ -10,17 +10,17 @@
         <xacro:ocean />
         <!--WAYPOINT OBJECT-->
-        <include>
+       <!--  <include>
             <name>wayPointMarker</name>
-            <pose>100.0 0.0 0 0 0 0</pose>
+            <pose>50 0.0 0 0 0 0</pose>
             <uri>$(find eboat_description)/models/wayPointMarker</uri>
         </include>
         <include>
             <name>buoy_red</name>
-            <pose>15 5 0 0 0 0 0</pose>
+            <pose>35 5 0 0 0 0 0</pose>
             <uri>$(find eboat_description)/models/buoy_red</uri>
         </include>
         <include>
             <name>buoy_green</name>
-            <pose>15.0 0.0 0 0 0 0 0</pose>
+            <pose>35 0.0 0 0 0 0 0</pose>
             <uri>$(find eboat_description)/models/buoy_green</uri>
         </include>
@@ -29,5 +29,5 @@
             <pose>-20.0 10.0 0 0 0 0 0</pose>
             <uri>$(find eboat_description)/models/buoy_yellow</uri>
-        </include>
+        </include> -->
         <!--PHYSICS ENGINE-->
         <physics type="ode">
@@ -38,5 +38,5 @@
             </ode>
             <max_step_size>0.01</max_step_size>
-            <real_time_update_rate>30</real_time_update_rate>
+            <real_time_update_rate>3000</real_time_update_rate>
         </physics>
     </world>
