Commit message: Working on esailor capabilities to sail just using wind. First esailor succeeded in sailing in close reach.

File: eboat_description/urdf/eboat4_control_plugins.xacro (robot description, xacro)
@@ -28,5 +28,5 @@
                 <link_name>base_link</link_name>
                 <way_point>wayPointMarker</way_point>
-                <frequency>3</frequency>
+                <frequency>1</frequency>
                 <propulsor_joint_name>propeller_joint</propulsor_joint_name>
             </plugin>

File: eboat_description/urdf/eboat4_physics_plugins.xacro (robot description, xacro)
@@ -1,4 +1,30 @@
 <?xml version="1.0"?>
 <robot xmlns:xacro="http://ros.org/wiki/xacro">
+    <!---->
+    <xacro:macro name="rudder_lift_drag" params="name">
+        <gazebo>
+            <plugin name="underwaterliftdrag_${name}" filename="libUnderWaterLiftDrag.so">
+                <link_name>rudder_link</link_name>
+                <forward>1 0 0</forward>
+                <upward>0 1 0</upward>
+                <area>0.19895</area>    <!--(m^2)-->
+                <cp>0 0 0</cp>
+                <water_density>997.0</water_density> <!--(kg/m^3)-->
+            </plugin>
+        </gazebo>
+    </xacro:macro>
+    <xacro:macro name="keel_lift_drag" params="name">
+        <gazebo>
+            <plugin name="underwaterliftdrag_${name}" filename="libUnderWaterLiftDrag.so">
+                <link_name>keel_link</link_name>
+                <forward>1 0 0</forward>
+                <upward>0 1 0</upward>
+                <area>0.48299</area>    <!--(m^2)-->
+                <cp>0 0 0</cp>
+                <water_density>997.0</water_density> <!--(kg/m^3)-->
+            </plugin>
+        </gazebo>
+    </xacro:macro>
+    <!---->
     <!--FOILS DYNAMICS USING LIFT AND DRAG (RUDDER, KEEL AND SAIL)-->
     <xacro:macro name="eboat_foil_gazebo" params="name">
@@ -13,9 +39,13 @@
                 <boom_joint_name>boom_joint</boom_joint_name>
                 <sail_cp>-0.012 0 1.5</sail_cp>
+                <!--<sail_cp>0.5 0 1.2</sail_cp>-->
+                <!--<sail_cp>0 0 1.2</sail_cp>-->
                 <rudder_link_name>rudder_link</rudder_link_name>
                 <rudder_forward>1 0 0</rudder_forward>
                 <rudder_upward>0 0 1</rudder_upward>
-                <rudder_area>0.1989</rudder_area>    <!--(m^2)-->
+                <rudder_area>0.10064</rudder_area>    <!--(m^2)-->
                 <rudder_cp>0 0 0</rudder_cp>
+                <keel_area>0.23779</keel_area>        <!--(m^2)-->
+                <keel_cp>0 0 0</keel_cp>
                 <water_density>997.0</water_density> <!--(kg/m^3)-->
             </plugin>
@@ -55,11 +85,13 @@
         <xU>${0.1 * 51.3}</xU>
         <xUU>${0.1 * 72.4}</xUU>
-        <yV>${0.2 * 80.0}</yV>
-        <yVV>${0.2 * 1600.0}</yVV>
+        <yV>${0.3 * 80.0}</yV>
+        <yVV>${0.3 * 1600.0}</yVV>
         <zW>${0.5 * 500.0}</zW>
         <zWW>0.0</zWW>
         <kP>${0.5 * 50.0}</kP>
         <mQ>${0.5 * 50.0}</mQ>
-        <nR>${0.15 * 400.0}</nR>
+        <!--<nR>${0.15 * 400.0}</nR>
+        <nRR>0.0</nRR>-->
+        <nR>${0.3 * 400.0}</nR>
         <nRR>0.0</nRR>
         <!-- General dimensions -->

File: eboat_description/urdf/eboat4tr.urdf.xacro (robot description, xacro)
@@ -17,4 +17,7 @@
     <!-- Attach lift&drag plugin for sail -->
     <xacro:eboat_foil_gazebo name="eboat4_sail"/>
+    <!-- Attach lift & drag plugin for uderwater elements -->
+    <!--<xacro:rudder_lift_drag name="rudder"/>-->
+    <!--<xacro:keel_lift_drag name="keel"/>-->
     <!--control interfaces-->
     <xacro:mission_control name="eboat4" />

File: eboat_gazebo/worlds/ocean.world.xacro (robot description, xacro)
@@ -5,4 +5,6 @@
           <camera name='user_camera'>
             <pose>-85.03 -3.517 26.21 0 0.212 -0.0332</pose>
+            <!--<pose>61.17 -7.023 4.735 0 0.208 3.0301</pose>-->
+            <!--<pose>61.96 -2.356 3.43 0 0.16 3.03</pose>-->
           </camera>
       </gui>
@@ -15,9 +17,9 @@
             <uri>$(find eboat_description)/models/wayPointMarker</uri>
         </include>-->
-        <!--<include>
+        <include>
             <name>redBuoy</name>
-            <pose>110.0 5.0 0 0 0 0</pose>
+            <pose>10.0 0 0 0 0 0</pose>
             <uri>$(find eboat_description)/models/buoy_red</uri>
-        </include>-->
+        </include>
         <!--PHYSICS ENGINE-->
         <physics type="ode">

File: eboat_gazebo/worlds/ocean_fixed_cam.world.xacro (robot description, xacro)
@@ -8,5 +8,6 @@
                     <static>true</static>
                     <use_model_frame>true</use_model_frame>
-                    <xyz>-30 0 8</xyz>
+                    <!--<xyz>-18 0 5</xyz>-->
+                    <xyz>-10.8 -6.44 2.5</xyz>
                     <!--<xyz>-15 0 4</xyz>-->
                     <inherit_yaw>true</inherit_yaw>

Commit message: Stable version for training PPO and SAC agents with EBoat53-v0.

File: eboat_description/urdf/eboat4_control_plugins.xacro (robot description, xacro)
@@ -28,5 +28,5 @@
                 <link_name>base_link</link_name>
                 <way_point>wayPointMarker</way_point>
-                <frequency>1</frequency>
+                <frequency>2</frequency>
                 <propulsor_joint_name>propeller_joint</propulsor_joint_name>
             </plugin>

File: eboat_description/urdf/eboat4tr.urdf.xacro (robot description, xacro)
@@ -233,11 +233,11 @@
         </inertial>
     </link>
-    <joint name="propeller_joint" type="revolute">
-        <origin xyz="-0.089683 -7.7043e-18 -0.949" rpy="-1.26162e-16 -0 0" />
+    <joint name="propeller_joint" type="continuous">
+        <origin xyz="-0.089683 0 -0.949" rpy="0 0 0" />
         <parent link="eletric_engine_link" />
         <child link="propeller_link" />
         <axis xyz="1 0 0"/>
         <limit effort="1000" velocity="20" />
-        <joint_properties friction="0.0"/>
+        <dynamics damping="0.0" friction="0.0"/>
     </joint>
     <link name="deck_link">

File: eboat_description/urdf/eboat4trOD.urdf.xacro (robot description, xacro)
@@ -26,6 +26,6 @@
     <xacro:propulsor_control_interface name="eboat4" />
     <!--RAY SENSOR-->
-    <gazebo reference="hokuyo_link">
-        <sensor type="gpu_ray" name="head_hokuyo_sensor">
+    <gazebo reference="camera_link">
+        <sensor type="ray" name="head_hokuyo_sensor">
             <pose>0 0 0 0 0 0</pose>
             <visualize>true</visualize>
@@ -34,14 +34,14 @@
                 <scan>
                 <horizontal>
-                    <samples>720</samples>
+                    <samples>121</samples>
                     <resolution>1</resolution>
-                    <min_angle>-1.570796</min_angle>
-                    <max_angle>1.570796</max_angle>
+                    <min_angle>-1.05</min_angle>
+                    <max_angle>1.05</max_angle>
                 </horizontal>
                 </scan>
                 <range>
-                <min>0.10</min>
-                <max>30.0</max>
-                <resolution>0.01</resolution>
+                <min>0.1</min>
+                <max>60.0</max>
+                <resolution>0.1</resolution>
                 </range>
                 <noise>
@@ -55,7 +55,7 @@
                 </noise>
             </ray>
-            <plugin name="gazebo_ros_head_hokuyo_controller" filename="libgazebo_ros_gpu_laser.so">
+            <plugin name="gazebo_ros_head_hokuyo_controller" filename="libgazebo_ros_laser.so">
                 <topicName>/eboat/laser/scan</topicName>
-                <frameName>camera_bow_link</frameName>
+                <frameName>camera_link</frameName>
             </plugin>
         </sensor>
@@ -269,5 +269,5 @@
         </inertial>
     </link>
-    <joint name="propeller_joint" type="revolute">
+    <joint name="propeller_joint" type="continuous">
         <origin xyz="-0.089683 -7.7043e-18 -0.949" rpy="-1.26162e-16 -0 0" />
         <parent link="eletric_engine_link" />
@@ -332,4 +332,20 @@
         <parent link="hull_link" />
         <child link="camera_bow_link" />
+    </joint>
+    <link name="camera_link">
+        <visual>
+        <origin xyz="0 0 0" rpy="0 1.5708 0" />
+        <!--<geometry>
+            <cylinder length="0.02" radius="0.02"/>
+        </geometry>-->
+        <!--<material name="camera_bow_material">
+            <color rgba="1.0 1.0 1.0 1.0"/>
+        </material>-->
+        </visual>
+    </link>
+    <joint name="camera_joint" type="fixed">
+        <origin xyz="${2.03098+0.180448} 0 ${0.645+0.125}" rpy="0 0 0" />
+        <parent link="deck_link" />
+        <child link="camera_link" />
     </joint>
     <!--COLORS-->

File: eboat_gazebo/worlds/ocean.world.xacro (robot description, xacro)
@@ -21,4 +21,9 @@
             <pose>10.0 0 0 0 0 0</pose>
             <uri>$(find eboat_description)/models/buoy_red</uri>
+        </include>
+        <include>
+            <name>yacht</name>
+            <pose>100.0 0 0 0 0 0</pose>
+            <uri>$(find eboat_description)/models/sailyacht</uri>
         </include>
         <!--PHYSICS ENGINE-->

File: eboat_gazebo/worlds/ocean.xacro (robot description, xacro)
@@ -32,4 +32,5 @@
     <!--WAVES-->
     <xacro:include filename="$(find wave_gazebo)/world_models/ocean_waves/model.xacro"/>
-    <xacro:ocean_waves scale="2.5"/>
+    <!--<xacro:ocean_waves scale="2.5"/>-->
+    <xacro:ocean_waves scale="3.5" gain="0.2" direction_x="0" direction_y="1"/>
 </world>
