Commit message: first stable version with gymnasium

File: eboat_description/urdf/eboat4.urdf.xacro (robot description, xacro)
@@ -7,5 +7,5 @@
                 <origin xyz="${xyz}" rpy="${rpy}" />
                 <geometry>
-                <mesh filename="package://eboat_description/models/eboat/meshes/${name}.stl"/>
+                <mesh filename="package://eboat_description/models/eboat4/meshes/${name}.stl"/>
                 </geometry>
             </visual>
@@ -24,5 +24,5 @@
                 <origin xyz="${xyz}" rpy="${rpy}" />
                 <geometry>
-                <mesh filename="package://eboat_description/models/eboat/meshes/support_hack_${name}.stl"/>
+                <mesh filename="package://eboat_description/models/eboat4/meshes/support_hack_${name}.stl"/>
                 </geometry>
                 <material name="support_hack_${name}_material">

File: fortune612_description/urdf/fortune612.urdf.xacro (robot description, xacro)
@@ -400,8 +400,18 @@
     </gazebo>
     <!--CONTROL LOOP INTERFACE-->
-    <gazebo>
+    <!--<gazebo>
         <plugin name="ctrl_loop" filename="libControlLoopPlugin.so">
             <frequency>1</frequency>
         </plugin>
+    </gazebo>-->
+    <gazebo>
+        <plugin name="rudder_control_interface_boto" filename="libRudderControllerPlugin.so">
+        <rudder_joint_name>rudder_joint</rudder_joint_name>
+        </plugin>
+    </gazebo>
+    <gazebo>
+        <plugin name="sail_control_interface_boto" filename="libSailControllerPlugin.so">
+            <sail_joint_name>boom_main_joint</sail_joint_name>
+        </plugin>
     </gazebo>
     <!--COLORS-->

Commit message: Feat: Lidar

File: eboat_description/urdf/eboat4.urdf.xacro (robot description, xacro)
@@ -180,4 +180,52 @@
         <child link="rope_c_link" />
     </joint>
+        <!-- Define a link for the LIDAR sensor -->
+    <link name="lidar_link">
+        <visual>
+        <origin xyz="0 0 0" rpy="0 0 0"/>
+        <geometry>
+            <cylinder length="0.1" radius="0.05"/>
+        </geometry>
+        <material name="Blue"/>
+        </visual>
+        <collision>
+        <origin xyz="0 0 0" rpy="0 0 0"/>
+        <geometry>
+            <cylinder length="0.1" radius="0.05"/>
+        </geometry>
+        </collision>
+    </link>
+    <!-- Attach the LIDAR sensor to the boat -->
+    <joint name="lidar_joint" type="fixed">
+        <parent link="base_link"/>
+        <child link="lidar_link"/>
+        <origin xyz="1 0 0.5" rpy="0 0 0"/>
+    </joint>
+    <!-- Add a Gazebo plugin to simulate the LIDAR sensor -->
+    <gazebo reference="lidar_link">
+        <sensor type="ray" name="lidar">
+        <always_on>true</always_on>
+        <update_rate>10</update_rate>
+        <ray>
+            <scan>
+            <horizontal>
+                <samples>720</samples>
+                <resolution>1</resolution>
+                <min_angle>-1.570796</min_angle>
+                <max_angle>1.570796</max_angle>
+            </horizontal>
+            </scan>
+            <range>
+            <min>0.08</min>
+            <max>10</max>
+            <resolution>0.01</resolution>
+            </range>
+            </ray>
+            <plugin name="gazebo_ros_head_hokuyo_controller" filename="libgazebo_ros_laser.so">
+            <topicName>/eboat/lidar</topicName>
+            <frameName>lidar_link</frameName>
+            </plugin>
+        </sensor>
+    </gazebo>
     <link name="keel_link">
         <visual>

Commit message: Last updates aiming for autonomous sailing agent. A image processing using opencv was included, but it has not been used on training yet.

File: eboat_description/urdf/eboat4.urdf.xacro (robot description, xacro)
@@ -149,10 +149,10 @@
     </link>
     <joint name="boom_joint" type="revolute">
-        <origin xyz="-0.049 -2.14313e-18 0.933" rpy="0 -0 0" />
+        <origin xyz="-0.049 0.0 0.933" rpy="0 0 0" />
         <parent link="mast_link" />
         <child link="boom_link" />
         <axis xyz="0 0 1"/>
         <limit effort="1000" velocity="5" lower="-1.5708" upper="1.5708"/>
-        <dynamics damping="2.0" friction="0.0"/>
+        <dynamics damping="0.5" friction="0.0"/>
     </joint>
     <link name="sail_link">

File: eboat_description/urdf/eboat4_physics_plugins.xacro (robot description, xacro)
@@ -16,7 +16,7 @@
                 <rudder_forward>1 0 0</rudder_forward>
                 <rudder_upward>0 0 1</rudder_upward>
-                <rudder_area>0.2</rudder_area>
+                <rudder_area>0.1989</rudder_area>    <!--(m^2)-->
                 <rudder_cp>0 0 0</rudder_cp>
-                <water_density>997.0</water_density>
+                <water_density>997.0</water_density> <!--(kg/m^3)-->
             </plugin>
         </gazebo>

File: eboat_gazebo/worlds/ocean.world.xacro (robot description, xacro)
@@ -2,7 +2,24 @@
 <sdf version="1.6" xmlns:xacro="http://ros.org/wiki/xacro">
     <world name="ocean">
+      <gui fullscreen='0'>
+          <camera name='user_camera'>
+            <pose>-85.03 -3.517 26.21 0 0.212 -0.0332</pose>
+          </camera>
+      </gui>
       <xacro:include filename="$(find eboat_gazebo)/worlds/ocean.xacro" />
       <xacro:ocean />
-      <physics type="ode">
+      <!--WAYPOINT OBJECT-->
+        <!--<include>
+            <name>wayPointMarker</name>
+            <pose>200.0 0.0 0 0 0 0</pose>
+            <uri>$(find eboat_description)/models/wayPointMarker</uri>
+        </include>-->
+        <!--<include>
+            <name>redBuoy</name>
+            <pose>110.0 5.0 0 0 0 0</pose>
+            <uri>$(find eboat_description)/models/buoy_red</uri>
+        </include>-->
+        <!--PHYSICS ENGINE-->
+        <physics type="ode">
           <ode>
               <solver>

File: eboat_gazebo/worlds/ocean_RL_training.world.xacro (robot description, xacro)
@@ -2,4 +2,9 @@
 <sdf version="1.6" xmlns:xacro="http://ros.org/wiki/xacro">
     <world name="ocean">
+        <gui fullscreen='0'>
+            <camera name='user_camera'>
+                <pose>-85.03 -3.517 26.21 0 0.212 -0.0332</pose>
+            </camera>
+        </gui>
         <xacro:include filename="$(find eboat_gazebo)/worlds/ocean.xacro" />
         <xacro:ocean />
@@ -7,5 +12,5 @@
         <include>
             <name>wayPointMarker</name>
-            <pose>0 100.0 0 0 0 0</pose>
+            <pose>100.0 0.0 0 0 0 0</pose>
             <uri>$(find eboat_description)/models/wayPointMarker</uri>
         </include>
