Commit message: Feat: dinamics

File: eboat_description/urdf/eboat4.urdf.xacro (robot description, xacro)
@@ -2,55 +2,19 @@
 <robot name="eboat4" xmlns:xacro="http://ros.org/wiki/xacro">
     <!--MACROS-->
-    <xacro:macro name="visual_link" params="name xyz rpy">
-        <link name="${name}_link">
-            <visual>
-                <origin xyz="${xyz}" rpy="${rpy}" />
-                <geometry>
-                <mesh filename="package://eboat_description/models/eboat4/meshes/${name}.stl"/>
-                </geometry>
-            </visual>
-        </link>
+    <xacro:macro name="support_hack" params="name xyz rpy">
+        <visual>
+            <origin xyz="${xyz}" rpy="${rpy}" />
+            <geometry>
+                <mesh filename="package://eboat_description/models/eboat4/meshes/support_hack_${name}.stl"/>
+            </geometry>
+        </visual>
     </xacro:macro>
-    <xacro:macro  name="rope_joints" params="name parent child xyz rpy">
-        <joint name="${name}_joint" type="fixed">
-            <origin xyz="${xyz}" rpy="${rpy}" />
-            <parent link="${parent}" />
-            <child link="${child}" />
-        </joint>
-    </xacro:macro>
-    <xacro:macro name="support_hack" params="name xyz rpy">
-        <link name="support_hack_${name}_link">
-            <visual>
-                <origin xyz="${xyz}" rpy="${rpy}" />
-                <geometry>
-                <mesh filename="package://eboat_description/models/eboat4/meshes/support_hack_${name}.stl"/>
-                </geometry>
-                <material name="support_hack_${name}_material">
-                <color rgba="0 0 0 1.0"/>
-                </material>
-            </visual>
-            <inertial>
-                <origin xyz="0 0 0" rpy="0 0 0"/>
-                <mass value="0" />
-                <inertia ixx="0" ixy="0"  ixz="0" iyy="0" iyz="0" izz="0" />
-            </inertial>
-        </link>
-    </xacro:macro>
-    <xacro:macro name="support_hack_joint" params="name xyz rpy">
-        <joint name="support_hack_${name}_joint" type="fixed">
-            <origin xyz="${xyz}" rpy="${rpy}" />
-            <parent link="deck_link" />
-            <child link="support_hack_${name}_link" />
-        </joint>
-    </xacro:macro>
+    <xacro:property name="mlength" value="${0.45+2.9+0.2}"/> <!--set the length of the main sail mast-->
     <xacro:include filename="$(find eboat_description)/urdf/eboat4_control_plugins.xacro"/>
     <xacro:include filename="$(find eboat_description)/urdf/eboat4_physics_plugins.xacro"/>
-    <xacro:property name="mlength" value="${0.45+2.9+0.2}"/> <!--set the length of the main sail mast-->
     <!-- Attach hydrodynamics plugin -->
     <xacro:usv_dynamics_gazebo name="eboat4_dynamics_plugin"/>
     <!-- Attach lift&drag plugin for sail -->
     <xacro:eboat_foil_gazebo name="eboat4_sail"/>
-    <!-- Attach lift&drag plugin for the wind vane -->
-    <xacro:eboat_windvane_gazebo name="eboat4_windvane"/>
     <!--control interfaces-->
     <xacro:mission_control name="eboat4" />
@@ -70,39 +34,43 @@
     <link name="hull_link">
         <visual>
-            <origin xyz="-1.24471 1.33227e-15 0.199376" rpy="0 -0 0" />
-            <geometry>
-                <mesh filename="package://eboat_description/models/eboat4/meshes/hull_link.dae"/>
-            </geometry>
-        </visual>
-        <collision>
-            <origin xyz="-0.1 0 0.214059" rpy="0 -0 0" />
+            <origin xyz="-1.23971 5.55112e-16 0.214059" rpy="0 -0 0" />
+            <geometry>
+                <mesh filename="package://eboat_description/models/eboat4/meshes/hull_link.stl"/>
+            </geometry>
+        </visual>
+        <collision>
+            <origin xyz="-1.23971 5.55112e-16 0.214059" rpy="0 -0 0" />
             <geometry>
                 <box size="2.7 1.0 0.63"/>
             </geometry>
         </collision>
-        <inertial>
-            <origin xyz="-0.198002 3.41823e-05 -0.0601847" rpy="0 0 0"/>
-            <mass value="83.6871" />
-            <inertia ixx="7.79423" ixy="-0.000716745"  ixz="1.26709" iyy="42.8173" iyz="-0.00040264" izz="47.1467" />
-        </inertial>
-    </link>
-    <link name="bow_link">
-        <visual>
-            <origin xyz="-2.48942 0 0.19871" rpy="0 -0 0" />
+        <!--ESPUMA -->
+        <visual>
+            <origin xyz="-1.23971 6.66134e-16 0.214073" rpy="0 -0 0" />
+            <geometry>
+                <mesh filename="package://eboat_description/models/eboat4/meshes/espuma.stl"/>
+            </geometry>
+        </visual>
+        <!--BOW-->
+        <visual>
+            <origin xyz="-1.23971 5.55112e-16 0.214059" rpy="0 -0 0" />
             <geometry>
                 <mesh filename="package://eboat_description/models/eboat4/meshes/bow_link.stl"/>
             </geometry>
         </visual>
-        <inertial>
-            <origin xyz="0.0248668 3.43326e-08 0.0804057" rpy="0 0 0"/>
-            <mass value="1.09744" />
-            <inertia ixx="0.00961813" ixy="9.91294e-09"  ixz="-0.000631055" iyy="0.00934886" iyz="-3.13957e-09" izz="0.000977479" />
-        </inertial>
-    </link>
-    <joint name="bow_joint" type="fixed">
-        <origin xyz="1.24471 0 0.000666379" rpy="0 0 0" />
-        <parent link="hull_link" />
-        <child link="bow_link" />
-    </joint>
+        <!--ELECTRIC ENGINE BASE-->
+        <visual>
+            <origin xyz="-1.23971 5.55112e-16 0.214059" rpy="0 -0 0" />
+            <geometry>
+                <mesh filename="package://eboat_description/models/eboat4/meshes/eletric_engine_base.stl"/>
+            </geometry>
+        </visual>
+        <!--INERTIA MATRIX-->
+        <inertial>
+            <origin xyz="-0.186398 3.25865e-05 -0.0426582" rpy="0 0 0"/>
+            <mass value="87.6741" />
+            <inertia ixx="8.07275" ixy="-0.000700071"  ixz="1.41913" iyy="47.1122" iyz="-0.000393928" izz="51.3333" />
+        </inertial>
+    </link>
     <link name="mast_link">
         <visual>
@@ -124,9 +92,4 @@
         </inertial>
     </link>
-    <joint name="mast_joint" type="fixed">
-        <origin xyz="0.59529 6.68277e-16 -0.153011" rpy="0 -0 0" />
-        <parent link="hull_link" />
-        <child link="mast_link" />
-    </joint>
     <link name="boom_link">
         <visual>
@@ -148,4 +111,22 @@
         </inertial>
     </link>
+    <link name="sail_link">
+        <visual>
+            <origin xyz="1.75893 -0.0664151 0" rpy="-1.5708 -0 0" />
+            <geometry>
+                <mesh filename="package://eboat_description/models/eboat4/meshes/sail.stl"/>
+            </geometry>
+        </visual>
+        <inertial>
+            <origin xyz="1.10322 1.09346 -1.24505e-20" rpy="0 0 0"/>
+            <mass value="2.216" />
+            <inertia ixx="1.15797" ixy="0.243689"  ixz="0" iyy="0.386027" iyz="0" izz="1.544" />
+        </inertial>
+    </link>
+    <joint name="sail_joint" type="fixed">
+        <origin xyz="-1.78373 0 0.0664151" rpy="1.5708 -0 0" />
+        <parent link="boom_link" />
+        <child link="sail_link" />
+    </joint>
     <joint name="boom_joint" type="revolute">
         <origin xyz="-0.049 -2.14313e-18 0.933" rpy="0 -0 0" />
@@ -156,76 +137,9 @@
         <dynamics damping="2.0" friction="0.0"/>
     </joint>
-    <link name="sail_link">
-        <visual>
-            <origin xyz="1.75893 -0.0664151 0" rpy="-1.5708 -0 0" />
-            <geometry>
-                <mesh filename="package://eboat_description/models/eboat4/meshes/sail.stl"/>
-            </geometry>
-        </visual>
-        <inertial>
-            <origin xyz="1.10322 1.09346 -1.24505e-20" rpy="0 0 0"/>
-            <mass value="2.216" />
-            <inertia ixx="1.15797" ixy="0.243689"  ixz="0" iyy="0.386027" iyz="0" izz="1.544" />
-        </inertial>
-    </link>
-    <xacro:visual_link name="rope_a" xyz="0.01 -2.636 0" rpy="-1.5708 0 0" />
-    <xacro:visual_link name="rope_b" xyz="0.01 -0.066 0" rpy="-1.5708 0 0" />
-    <xacro:visual_link name="rope_c" xyz="1.773 -0.0223 0" rpy="-1.5708 0 0" />
-    <xacro:rope_joints name="rope_a" parent="sail_link" child="rope_a_link" xyz="1.74893 2.56958 0" rpy="0 0 0" />
-    <xacro:rope_joints name="rope_b" parent="sail_link" child="rope_b_link" xyz="1.74893 -0.000415051 0" rpy="0 0 0" />
-    <xacro:rope_joints name="rope_c" parent="rope_c_link" child="sail_link" xyz="0.0140742 0.0441151 0" rpy="0 0 0" />
-    <joint name="sail_joint_2" type="fixed">
-        <origin xyz="-1.7978 0 0.0223" rpy="1.5708 0 0" />
-        <parent link="boom_link" />
-        <child link="rope_c_link" />
-    </joint>
-        <!-- Define a link for the LIDAR sensor -->
-    <link name="lidar_link">
-        <visual>
-        <origin xyz="0 0 0" rpy="0 0 0"/>
-        <geometry>
-            <cylinder length="0.5" radius="0.05"/>
-        </geometry>
-        <material name="Blue"/>
-        </visual>
-        <collision>
-        <origin xyz="0 0 0" rpy="0 0 0"/>
-        <geometry>
-            <cylinder length="0.5" radius="0.05"/>
-        </geometry>
-        </collision>
-    </link>
-    <!-- Attach the LIDAR sensor to the boat -->
-    <joint name="lidar_joint" type="fixed">
-        <parent link="base_link"/>
-        <child link="lidar_link"/>
-        <origin xyz="1 0 0.5" rpy="0 0 0"/>
-    </joint>
-    <!-- Add a Gazebo plugin to simulate the LIDAR sensor -->
-    <gazebo reference="lidar_link">
-        <sensor type="ray" name="lidar">
-        <always_on>true</always_on>
-        <update_rate>10</update_rate>
-        <ray>
-            <scan>
-            <horizontal>
-                <samples>720</samples>
-                <resolution>1</resolution>
-                <min_angle>-1.570796</min_angle>
-                <max_angle>1.570796</max_angle>
-            </horizontal>
-            </scan>
-            <range>
-            <min>0.08</min>
-            <max>10</max>
-            <resolution>0.01</resolution>
-            </range>
-            </ray>
-            <plugin name="gazebo_ros_head_hokuyo_controller" filename="libgazebo_ros_laser.so">
-            <topicName>/eboat/lidar</topicName>
-            <frameName>lidar_link</frameName>
-            </plugin>
-        </sensor>
-    </gazebo>
+    <joint name="mast_joint" type="fixed">
+        <origin xyz="0.59529 6.68277e-16 -0.153011" rpy="0 -0 0" />
+        <parent link="hull_link" />
+        <child link="mast_link" />
+    </joint>
     <link name="keel_link">
         <visual>
@@ -282,22 +196,4 @@
         <dynamics damping="0.0" friction="2.0"/>
     </joint>
-    <link name="eletric_engine_base_link">
-        <visual>
-            <origin xyz="0 0 0" rpy="0 -0 0" />
-            <geometry>
-                <mesh filename="package://eboat_description/models/eboat4/meshes/eletric_engine_base.stl"/>
-            </geometry>
-        </visual>
-        <inertial>
-            <origin xyz="-0.0177716 0 0.122132" rpy="0 0 0"/>
-            <mass value="0.887162" />
-            <inertia ixx="0.0037743" ixy="0"  ixz="0.000214551" iyy="0.00311449" iyz="0" izz="0.00287765" />
-        </inertial>
-    </link>
-    <joint name="eletric_egine_base" type="fixed">
-        <origin xyz="-1.24471 0 0.199376" rpy="0 0 0" />
-        <parent link="hull_link" />
-        <child link="eletric_engine_base_link" />
-    </joint>
     <link name="eletric_engine_link">
         <visual>
@@ -334,120 +230,49 @@
         </inertial>
     </link>
-    <joint name="propeller_joint" type="continuous">
+    <joint name="propeller_joint" type="revolute">
         <origin xyz="-0.089683 -7.7043e-18 -0.949" rpy="-1.26162e-16 -0 0" />
         <parent link="eletric_engine_link" />
         <child link="propeller_link" />
-        <axis xyz="1 0 0"/>
-        <limit effort="1000" velocity="20" />
-        <dynamics damping="0.0" friction="0.0"/>
-    </joint>
-    <link name="biruta_link">
-        <visual>
-            <origin xyz="-0.161823 -5.20475e-19 -2.832" rpy="0 -0 0" />
-            <geometry>
-                <mesh filename="package://eboat_description/models/eboat4/meshes/biruta.stl"/>
-            </geometry>
-        </visual>
-        <inertial>
-            <origin xyz="-0.0148129 1.0796e-10 0.0419007" rpy="0 0 0"/>
-            <mass value="0.0021539" />
-            <inertia ixx="1.19286e-06" ixy="-1.19699e-14"  ixz="6.09373e-07" iyy="2.92342e-06" iyz="-4.59008e-15" izz="1.8198e-06" />
-        </inertial>
-    </link>
-    <joint name="biruta_joint" type="continuous">
-        <origin xyz="0.161823 -2.14313e-18 3.765" rpy="0 -0 0" />
-        <parent link="mast_link" />
-        <child link="biruta_link" />
         <axis xyz="0 0 1"/>
-        <limit effort="1" velocity="2"/>
-        <dynamics damping="0.0" friction="0.00002"/>
-    </joint>
-    <link name="camera_top_link">
-        <visual>
-            <origin xyz="0.053 0 -2.832" rpy="0 -0 0" />
-            <geometry>
-                <mesh filename="package://eboat_description/models/eboat4/meshes/camera_top.stl"/>
-            </geometry>
-        </visual>
-        <inertial>
-            <origin xyz="0 0 0" rpy="0 0 0"/>
-            <mass value="0" />
-            <inertia ixx="0" ixy="0"  ixz="0" iyy="0" iyz="0" izz="0" />
-        </inertial>
-    </link>
-    <joint name="camera_top_joint" type="fixed">
-        <origin xyz="-0.053 0 3.765" rpy="0 0 0" />
-        <parent link="mast_link" />
-        <child link="camera_top_link" />
+        <limit effort="1" velocity="20" />
+        <joint_properties friction="0.0"/>
     </joint>
     <link name="deck_link">
         <visual>
             <origin xyz="0 0 0" rpy="0 0 0" />
-                <geometry>
+            <geometry>
             <mesh filename="package://eboat_description/models/eboat4/meshes/deck.stl"/>
             </geometry>
         </visual>
-        <inertial>
-            <origin xyz="1.10267 0.00505112 0.0298862" rpy="0 0 0"/>
-            <mass value="4.65558" />
-            <inertia ixx="0.384796" ixy="0.0209115"  ixz="0.00217436" iyy="1.95434" iyz="0.000402869" izz="2.33348" />
+        <xacro:support_hack name="port_1" xyz="0 0 0" rpy="0 0 0" />
+        <xacro:support_hack name="port_2" xyz="0 0 0" rpy="0 0 0" />
+        <xacro:support_hack name="port_3" xyz="0 0 0" rpy="0 0 0" />
+        <xacro:support_hack name="port_4" xyz="0 0 0" rpy="0 0 0" />
+        <xacro:support_hack name="starboard_1" xyz="0 0 0" rpy="0 0 0" />
+        <xacro:support_hack name="starboard_2" xyz="0 0 0" rpy="0 0 0" />
+        <xacro:support_hack name="starboard_3" xyz="0 0 0" rpy="0 0 0" />
+        <xacro:support_hack name="starboard_4" xyz="0 0 0" rpy="0 0 0" />
+        <visual>
+            <origin xyz="-4.44089e-16 1.11022e-16 5.55112e-17" rpy="0 -0 0" />
+            <geometry>
+            <mesh filename="package://eboat_description/models/eboat4/meshes/hack_starboard.stl"/>
+            </geometry>
+        </visual>
+        <visual>
+            <origin xyz="0 0 5.55112e-17" rpy="0 -0 0" />
+            <geometry>
+                <mesh filename="package://eboat_description/models/eboat4/meshes/hack_port.stl"/>
+            </geometry>
+        </visual>
+        <inertial>
+            <origin xyz="1.17098 0.0029352 0.08114" rpy="0 0 0"/>
+            <mass value="8.12081" />
+            <inertia ixx="0.940446" ixy="0.0228946"  ixz="-0.0360182" iyy="3.85004" iyz="0.00158452" izz="4.72607" />
         </inertial>
     </link>
     <joint name="deck_joint" type="fixed">
-        <origin xyz="-1.24471 0 0.199376" rpy="0 0 0" />
+        <origin xyz="-1.23971 5.55112e-16 0.214059" rpy="0 -0 0" />
         <parent link="hull_link" />
         <child link="deck_link" />
-    </joint>
-    <xacro:support_hack name="port_1" xyz="-0.0410859 -0.407092 -0.05" rpy="0 0 0" />
-    <xacro:support_hack_joint name="port_1" xyz="0.0410859 0.407092 0.05" rpy="0 0 0" />
-    <xacro:support_hack name="port_2" xyz="-0.776847 -0.466397 -0.05" rpy="0 0 0" />
-    <xacro:support_hack_joint name="port_2" xyz="0.776847 0.466397 0.05" rpy="0 0 0" />
-    <xacro:support_hack name="port_3" xyz="-1.58684 -0.364972 -0.05" rpy="0 0 0" />
-    <xacro:support_hack_joint name="port_3" xyz="1.58684 0.364972 0.05" rpy="0 0 0" />
-    <xacro:support_hack name="port_4" xyz="-2.44761 -0.0712925 -0.05" rpy="0 0 0" />
-    <xacro:support_hack_joint name="port_4" xyz="2.44761 0.0712925 0.05" rpy="0 0 0" />
-    <xacro:support_hack name="starboard_1" xyz="-0.0410859 0.407092 -0.05" rpy="0 0 0" />
-    <xacro:support_hack_joint name="starboard_1" xyz="0.0410859 -0.407092 0.05" rpy="0 0 0" />
-    <xacro:support_hack name="starboard_2" xyz="-0.776847 0.466397 -0.05" rpy="0 0 0" />
-    <xacro:support_hack_joint name="starboard_2" xyz="0.776847 -0.466397 0.05" rpy="0 0 0" />
-    <xacro:support_hack name="starboard_3" xyz="-1.58684 0.364972 -0.05" rpy="0 0 0" />
-    <xacro:support_hack_joint name="starboard_3" xyz="1.58684 -0.364972 0.05" rpy="0 0 0" />
-    <xacro:support_hack name="starboard_4" xyz="-2.44761 0.071293 -0.05" rpy="0 0 0" />
-    <xacro:support_hack_joint name="starboard_4" xyz="2.44761 -0.071293 0.05" rpy="0 0 0" />
-    <link name="hack_port_link">
-        <visual>
-            <origin xyz="-2.25991 0.14 -0.976456" rpy="1.5708 -0.372391 0" />
-            <geometry>
-                <mesh filename="package://eboat_description/models/eboat4/meshes/hack_port.stl"/>
-            </geometry>
-        </visual>
-        <inertial>
-            <origin xyz="-1.21877 -0.00999996 -0.172045" rpy="0 0 0"/>
-            <mass value="1.73299" />
-            <inertia ixx="0.145894" ixy="0.307705"  ixz="-0.11957" iyy="0.813431" iyz="0.0467072" izz="0.908646" />
-        </inertial>
-    </link>
-    <joint name="hack_port_joint" type="fixed">
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
File: eboat_description/urdf/eboat4tr.urdf.xacro (robot description, xacro)
@@ -303,8 +303,8 @@
             <material name="blue"/>
             </visual>
-            <inertial>
-            <origin xyz="0 0 0" rpy="0 0 0"/>
-            <mass value="0.1"/>
-            <inertia ixx="1.0" ixy="2.0" ixz="0" iyy="1.0" iyz="0" izz="1.0"/>
+           <inertial>
+                <origin xyz="0 0 0" rpy="0 0 0"/>
+                <mass value="0.1"/>
+                <inertia ixx="0.0001" ixy="0" ixz="0" iyy="0.0001" iyz="0" izz="0.0001"/>
             </inertial>
         </link>
@@ -317,4 +317,10 @@
     <!-- LIDAR Gazebo plugin -->
     <gazebo reference="lidar_link">
+           <material>Gazebo/Grey</material>
+            <contact>
+                <collide_without_contact>true</collide_without_contact>
+                <collide_bitmask>0x02</collide_bitmask>
+                <collide_without_contact_bitmask>0x01</collide_without_contact_bitmask>
+            </contact>
         <sensor type="ray" name="lidar">
             <pose>0 0 0 0 0 0</pose>

File: eboat_gazebo/worlds/ocean.xacro (robot description, xacro)
@@ -21,4 +21,19 @@
             <!--<heading_deg>180</heading_deg>-->
         </spherical_coordinates>
+        <physics type="ode">
+            <ode>
+                <solver>
+                    <type>quick</type>
+                    <iters>150</iters>
+                    <sor>1.3</sor>
+                </solver>
+                <constraints>
+                    <cfm>0.00001</cfm>
+                    <erp>0.2</erp>
+                    <contact_max_correcting_vel>100.0</contact_max_correcting_vel>
+                    <contact_surface_layer>0.001</contact_surface_layer>
+                </constraints>
+            </ode>
+        </physics>
         <!---->
         <gravity>0.0 0.0 -9.81</gravity>

File: eboat_gazebo/worlds/ocean_RL_training.world.xacro (robot description, xacro)
@@ -15,4 +15,14 @@
             <uri>$(find eboat_description)/models/buoy_red</uri>
         </include>
+        <include>
+            <name>buoy_green</name>
+            <pose>20 0 0 0 0 0 0</pose>
+            <uri>$(find eboat_description)/models/buoy_green</uri>
+        </include>
+        <include>
+            <name>buoy_yellow</name>
+            <pose>30 0 0 0 0 0 0</pose>
+            <uri>$(find eboat_description)/models/buoy_yellow</uri>
+        </include>
         <!--PHYSICS ENGINE-->
         <physics type="ode">
