Commit message: From now on, sensor plugins will be declared on eboat_description/urdf/eboat4_sensors_plugins.xacro

File: eboat_description/urdf/eboat4.urdf.xacro (robot description, xacro)
@@ -46,4 +46,5 @@
     <xacro:include filename="$(find eboat_description)/urdf/eboat4_control_plugins.xacro"/>
     <xacro:include filename="$(find eboat_description)/urdf/eboat4_physics_plugins.xacro"/>
+    <xacro:include filename="$(find eboat_description)/urdf/eboat4_sensors_plugins.xacro"/>
     <xacro:property name="mlength" value="${0.45+2.9+0.2}"/> <!--set the length of the main sail mast-->
     <!-- Attach hydrodynamics plugin -->
@@ -58,4 +59,7 @@
     <xacro:rudder_control_interface name="eboat4" />
     <xacro:propulsor_control_interface name="eboat4" />
+    <!--SENSORS-->
+    <xacro:bow_camera/>
+    <xacro:bow_beam_detector visualize="True"/>
     <!--ROBOT DESCRIPTION-->
     <link name="base_link">
@@ -581,79 +585,3 @@
         <material>Gazebo/BlueTransparent</material>
     </gazebo>
-    <!-- CAMERA -->
-    <gazebo reference="camera_link">
-        <sensor type="camera" name="bow_camera">
-        <update_rate>30.0</update_rate>
-        <camera name="head">
-            <horizontal_fov>1.3962634</horizontal_fov>
-            <image>
-            <width>800</width>
-            <height>800</height>
-            <format>R8G8B8</format>
-            </image>
-            <clip>
-            <near>0.02</near>
-            <far>300</far>
-            </clip>
-            <noise>
-            <type>gaussian</type>
-            <!-- Noise is sampled independently per pixel on each frame.
-                That pixel's noise value is added to each of its color
-                channels, which at that point lie in the range [0,1]. -->
-            <mean>0.0</mean>
-            <stddev>0.007</stddev>
-            </noise>
-        </camera>
-        <plugin name="camera_controller" filename="libgazebo_ros_camera.so">
-            <alwaysOn>true</alwaysOn>
-            <updateRate>0.0</updateRate>
-            <cameraName>mission_control/bow_camera</cameraName>
-            <imageTopicName>image_raw</imageTopicName>
-            <cameraInfoTopicName>camera_info</cameraInfoTopicName>
-            <frameName>camera_bow_link</frameName>
-            <hackBaseline>0.07</hackBaseline>
-            <distortionK1>0.0</distortionK1>
-            <distortionK2>0.0</distortionK2>
-            <distortionK3>0.0</distortionK3>
-            <distortionT1>0.0</distortionT1>
-            <distortionT2>0.0</distortionT2>
-        </plugin>
-        </sensor>
-    </gazebo>
-    <!--RAY SENSOR-->
-    <gazebo reference="camera_link">
-        <sensor type="ray" name="head_hokuyo_sensor">
-            <pose>0 0 0 0 0 0</pose>
-            <visualize>true</visualize>
-            <update_rate>40</update_rate>
-            <ray>
-                <scan>
-                <horizontal>
-                    <samples>121</samples>
-                    <resolution>1</resolution>
-                    <min_angle>-1.05</min_angle>
-                    <max_angle>1.05</max_angle>
-                </horizontal>
-                </scan>
-                <range>
-                <min>0.1</min>
-                <max>60.0</max>
-                <resolution>0.1</resolution>
-                </range>
-                <noise>
-                <type>gaussian</type>
-                <!-- Noise parameters based on published spec for Hokuyo laser
-                    achieving "+-30mm" accuracy at range < 10m.  A mean of 0.0m and
-                    stddev of 0.01m will put 99.7% of samples within 0.03m of the true
-                    reading. -->
-                <mean>0.0</mean>
-                <stddev>0.01</stddev>
-                </noise>
-            </ray>
-            <plugin name="gazebo_ros_head_hokuyo_controller" filename="libgazebo_ros_laser.so">
-                <topicName>/eboat/laser/scan</topicName>
-                <frameName>camera_link</frameName>
-            </plugin>
-        </sensor>
-    </gazebo>
 </robot>

File: eboat_description/urdf/eboat4trOD.urdf.xacro (robot description, xacro)
@@ -13,4 +13,5 @@
     <xacro:include filename="$(find eboat_description)/urdf/eboat4_control_plugins.xacro"/>
     <xacro:include filename="$(find eboat_description)/urdf/eboat4_physics_plugins.xacro"/>
+    <xacro:include filename="$(find eboat_description)/urdf/eboat4_sensors_plugins.xacro"/>
     <!-- Attach hydrodynamics plugin -->
     <xacro:usv_dynamics_gazebo name="eboat4_dynamics_plugin"/>
@@ -25,40 +26,6 @@
     <xacro:rudder_control_interface name="eboat4" />
     <xacro:propulsor_control_interface name="eboat4" />
-    <!--RAY SENSOR-->
-    <gazebo reference="camera_link">
-        <sensor type="ray" name="head_hokuyo_sensor">
-            <pose>0 0 0 0 0 0</pose>
-            <visualize>true</visualize>
-            <update_rate>40</update_rate>
-            <ray>
-                <scan>
-                <horizontal>
-                    <samples>121</samples>
-                    <resolution>1</resolution>
-                    <min_angle>-1.05</min_angle>
-                    <max_angle>1.05</max_angle>
-                </horizontal>
-                </scan>
-                <range>
-                <min>0.1</min>
-                <max>60.0</max>
-                <resolution>0.1</resolution>
-                </range>
-                <noise>
-                <type>gaussian</type>
-                <!-- Noise parameters based on published spec for Hokuyo laser
-                    achieving "+-30mm" accuracy at range < 10m.  A mean of 0.0m and
-                    stddev of 0.01m will put 99.7% of samples within 0.03m of the true
-                    reading. -->
-                <mean>0.0</mean>
-                <stddev>0.01</stddev>
-                </noise>
-            </ray>
-            <plugin name="gazebo_ros_head_hokuyo_controller" filename="libgazebo_ros_laser.so">
-                <topicName>/eboat/laser/scan</topicName>
-                <frameName>camera_link</frameName>
-            </plugin>
-        </sensor>
-    </gazebo>
+    <!--SENSORS-->
+    <xacro:bow_beam_detector visualize="False"/>
     <!--ROBOT DESCRIPTION-->
     <link name="base_link">
@@ -72,5 +39,5 @@
     </joint>
     <link name="hull_link">
-        <visual>
+        <visual name="hull_visual">
             <origin xyz="-1.23971 5.55112e-16 0.214059" rpy="0 -0 0" />
             <geometry>
@@ -78,5 +45,5 @@
             </geometry>
         </visual>
-        <collision>
+        <collision name="hull_collision">
             <origin xyz="-1.23971 5.55112e-16 0.214059" rpy="0 -0 0" />
             <geometry>

Commit message: Start implementing the contact sensor.

File: eboat_description/urdf/eboat4.urdf.xacro (robot description, xacro)
@@ -62,4 +62,5 @@
     <xacro:bow_camera/>
     <xacro:bow_beam_detector visualize="True"/>
+    <!--<xacro:contact_sensor>-->
     <!--ROBOT DESCRIPTION-->
     <link name="base_link">

File: eboat_description/urdf/eboat4_sensors_plugins.xacro (robot description, xacro)
@@ -79,3 +79,17 @@
         </gazebo>
     </xacro:macro>
+    <!--xacro:macro name="contact_sensor">
+        <gazebo reference="hull_link">
+            <sensor name="contactsensor_sensor" type="contact">
+                <always_on>true</always_on>
+                <contact>
+                    <collision>hull_collision</collision>
+                </contact>
+                <plugin filename="libgazebo_ros_bumper.so" name="left_arm_fist_plugin">
+                    <bumperTopicName>hull_contact</bumperTopicName>
+                    <frameName>hull_link</frameName>
+                </plugin>
+            </sensor>
+        </gazebo>
+    </xacro:macro>-->
 </robot>

File: eboat_description/urdf/eboat4trOD.urdf.xacro (robot description, xacro)
@@ -40,5 +40,5 @@
     <link name="hull_link">
         <visual name="hull_visual">
-            <origin xyz="-1.23971 5.55112e-16 0.214059" rpy="0 -0 0" />
+            <origin xyz="-1.23971 0 0.214059" rpy="0 0 0"/>
             <geometry>
                 <mesh filename="package://eboat_description/models/eboat4/meshes/hull_link.stl"/>

Commit message: The wind speed and angle, the boat position in the world frame, and the ahead direction are now published in individual ros topics.

File: eboat_description/urdf/eboat4.urdf.xacro (robot description, xacro)
@@ -55,5 +55,8 @@
     <xacro:eboat_windvane_gazebo name="eboat4_windvane"/>
     <!--control interfaces-->
-    <xacro:mission_control name="eboat4" />
+    <!--<xacro:mission_control name="eboat4" />-->
+    <xacro:wind_sensor name="eboat4" />
+    <xacro:bow_vector name="eboat4" />
+    <xacro:CPS name="eboat4" />
     <xacro:sail_control_interface name="eboat4" />
     <xacro:rudder_control_interface name="eboat4" />

File: eboat_description/urdf/eboat4_control_plugins.xacro (robot description, xacro)
@@ -33,3 +33,27 @@
         </gazebo>
     </xacro:macro>
+    <xacro:macro name="wind_sensor" params="name">
+        <gazebo>
+            <plugin name="wind_sensor_${name}" filename="libWindSensorPlugin.so">
+                <link_name>biruta_link</link_name>
+                <frequency>1</frequency>
+            </plugin>
+        </gazebo>
+    </xacro:macro>
+    <xacro:macro name="CPS" params="name">
+        <gazebo>
+            <plugin name="CPS_${name}" filename="libCPSPlugin.so">
+                <link_name>base_link</link_name>
+                <frequency>1</frequency>
+            </plugin>
+        </gazebo>
+    </xacro:macro>
+    <xacro:macro name="bow_vector" params="name">
+        <gazebo>
+            <plugin name="bow_vector_${name}" filename="libBowVectorPlugin.so">
+                <link_name>base_link</link_name>
+                <frequency>1</frequency>
+            </plugin>
+        </gazebo>
+    </xacro:macro>
 </robot>
